File: PCB/nixie-2/nixie-2.kicad_sch (KiCad schematic)
At the start: 2 parts

Commit message: Added files for a PCB
Parts:
- added U?: ARDUINO_PRO_MINI, MODULE_ARDUINO_PRO_MINI, symbol nixie-2-symbols:ARDUINO_PRO_MINI
Connections:
- new net: U?.JP1_5 (GND), U?.JP1_6 (GND)
Changed lines of the file:
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@@
     (stroke (width 0) (type default) (color 0 0 0 0))
+  )
+  (symbol (lib_id "nixie-2-symbols:ARDUINO_PRO_MINI") (at 163.83 67.31 0) (unit 1)
+    (in_bom yes) (on_board yes) (fields_autoplaced)
+    (property "Reference" "U?" (id 0) (at 163.83 31.75 0))
+    (property "Value" "ARDUINO_PRO_MINI" (id 1) (at 163.83 34.29 0))
+    (property "Footprint" "MODULE_ARDUINO_PRO_MINI" (id 2) (at 163.83 67.31 0)
+      (effects (font (size 1.27 1.27)) (justify left bottom) hide)
+    )
+    (property "Datasheet" "" (id 3) (at 163.83 67.31 0)
+      (effects (font (size 1.27 1.27)) (justify left bottom) hide)
+    )
+    (property "PARTREV" "N/A" (id 4) (at 163.83 67.31 0)
+      (effects (font (size 1.27 1.27)) (justify left bottom) hide)
+    )
+    (property "MANUFACTURER" "SparkFun Electronics" (id 5) (at 163.83 67.31 0)
+      (effects (font (size 1.27 1.27)) (justify left bottom) hide)
+    )
+    (property "MAXIMUM_PACKAGE_HEIGHT" "N/A" (id 6) (at 163.83 67.31 0)
+      (effects (font (size 1.27 1.27)) (justify left bottom) hide)
+    )
+    (property "STANDARD" "Manufacturer Recommendations" (id 7) (at 163.83 67.31 0)
+      (effects (font (size 1.27 1.27)) (justify left bottom) hide)
+    )
+    (pin "JP1_1")
+    (pin "JP1_2")
+    (pin "JP1_3")
+    (pin "JP1_4")
+    (pin "JP1_5")
+    (pin "JP1_6")
+    (pin "JP2_1")
+    (pin "JP2_2")
+    (pin "JP3_1")
+    (pin "JP3_2")
+    (pin "JP6_1")
+    (pin "JP6_10")
+    (pin "JP6_11")
+    (pin "JP6_12")
+    (pin "JP6_2")
+    (pin "JP6_3")
+    (pin "JP6_4")
+    (pin "JP6_5")
+    (pin "JP6_6")
+    (pin "JP6_7")
+    (pin "JP6_8")
+    (pin "JP6_9")
+    (pin "JP7_1")
+    (pin "JP7_10")
+    (pin "JP7_11")
+    (pin "JP7_12")
+    (pin "JP7_2")
+    (pin "JP7_3")
+    (pin "JP7_4")
+    (pin "JP7_5")
+    (pin "JP7_6")
+    (pin "JP7_7")
+    (pin "JP7_8")
+    (pin "JP7_9")
   )
   (symbol (lib_id "MUR160G:MUR160G") (at 116.84 66.04 0) (unit 1)
@@
       (reference "L1") (unit 1) (value "L_Ferrite") (footprint "Inductor_THT:L_Radial_D16.8mm_P12.07mm_Vishay_IHB-1")
     )
+    (path "/39cf93f6-4fc8-42ac-abab-83e65b5f03d5"
+      (reference "U?") (unit 1) (value "ARDUINO_PRO_MINI") (footprint "MODULE_ARDUINO_PRO_MINI")
+    )
   )
