File: PCB/nixie-2/nixie-2.kicad_sch (KiCad schematic)
At the start: 2 parts

Commit message: symbols and footprints
Parts:
- added V? (x3): Z57xM, symbol nixie-1:Z57xM
Changed lines of the file:
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@@
     (stroke (width 0) (type default) (color 0 0 0 0))
+  )
+  (symbol (lib_id "nixie-1:Z57xM") (at 147.32 107.95 0) (unit 1)
+    (in_bom yes) (on_board yes) (fields_autoplaced)
+    (property "Reference" "V?" (id 0) (at 164.465 105.2103 0)
+      (effects (font (size 1.27 1.27)) (justify left))
+    )
+    (property "Value" "Z57xM" (id 1) (at 164.465 107.7472 0)
+      (effects (font (size 1.27 1.27)) (justify left))
+    )
+    (property "Footprint" "" (id 2) (at 152.4 109.22 0)
+      (effects (font (size 1.524 1.524)))
+    )
+    (property "Datasheet" "" (id 3) (at 152.4 109.22 0)
+      (effects (font (size 1.524 1.524)))
+    )
+    (pin "1")
+    (pin "10")
+    (pin "11")
+    (pin "12")
+    (pin "13")
+    (pin "2")
+    (pin "3")
+    (pin "4")
+    (pin "5")
+    (pin "6")
+    (pin "7")
+    (pin "8")
+    (pin "9")
+  )
+  (symbol (lib_id "nixie-1:Z57xM") (at 195.58 107.95 0) (unit 1)
+    (in_bom yes) (on_board yes) (fields_autoplaced)
+    (property "Reference" "V?" (id 0) (at 212.725 105.2103 0)
+      (effects (font (size 1.27 1.27)) (justify left))
+    )
+    (property "Value" "Z57xM" (id 1) (at 212.725 107.7472 0)
+      (effects (font (size 1.27 1.27)) (justify left))
+    )
+    (property "Footprint" "" (id 2) (at 200.66 109.22 0)
+      (effects (font (size 1.524 1.524)))
+    )
+    (property "Datasheet" "" (id 3) (at 200.66 109.22 0)
+      (effects (font (size 1.524 1.524)))
+    )
+    (pin "1")
+    (pin "10")
+    (pin "11")
+    (pin "12")
+    (pin "13")
+    (pin "2")
+    (pin "3")
+    (pin "4")
+    (pin "5")
+    (pin "6")
+    (pin "7")
+    (pin "8")
+    (pin "9")
   )
   (symbol (lib_id "MUR160G:MUR160G") (at 116.84 66.04 0) (unit 1)
@@
     (pin "2")
   )
+  (symbol (lib_id "nixie-1:Z57xM") (at 96.52 107.95 0) (unit 1)
+    (in_bom yes) (on_board yes) (fields_autoplaced)
+    (property "Reference" "V?" (id 0) (at 113.665 105.2103 0)
+      (effects (font (size 1.27 1.27)) (justify left))
+    )
+    (property "Value" "Z57xM" (id 1) (at 113.665 107.7472 0)
+      (effects (font (size 1.27 1.27)) (justify left))
+    )
+    (property "Footprint" "" (id 2) (at 101.6 109.22 0)
+      (effects (font (size 1.524 1.524)))
+    )
+    (property "Datasheet" "" (id 3) (at 101.6 109.22 0)
+      (effects (font (size 1.524 1.524)))
+    )
+    (pin "1")
+    (pin "10")
+    (pin "11")
+    (pin "12")
+    (pin "13")
+    (pin "2")
+    (pin "3")
+    (pin "4")
+    (pin "5")
+    (pin "6")
+    (pin "7")
+    (pin "8")
+    (pin "9")
+  )
   (sheet_instances
     (path "/" (page "1"))
@@
       (reference "L1") (unit 1) (value "L_Ferrite") (footprint "Inductor_THT:L_Radial_D16.8mm_P12.07mm_Vishay_IHB-1")
     )
+    (path "/1f56af86-7df6-4c1e-88a4-993f39743e67"
+      (reference "V?") (unit 1) (value "Z57xM") (footprint "")
+    )
+    (path "/347ce5cd-8436-49a5-80d7-2b6bb580a593"
+      (reference "V?") (unit 1) (value "Z57xM") (footprint "")
+    )
+    (path "/fcee0de7-d38d-4323-aa93-a47d894a62af"
+      (reference "V?") (unit 1) (value "Z57xM") (footprint "")
+    )
   )
