File: PCB/Z573M-tube/Z573M-tube.kicad_pcb (KiCad board)
At the start: 2 copper layers, 20.3 x 29.2 mm, 3 parts, among them J1 6-pin-header, J2 6-pin-header

Commit message: New board, v 2.0, with gerber files
Parts:
- Version 2.0: renamed from V1; footprint nixie-footprints:Z57xM-v1 -> nixie-footprints:Z57xM-v3-HV
Routing:
- net /K5: track 9.11 -> 8.31 mm
- net /K6: track 8.44 -> 7.70 mm
- net /K4: track 10.8 -> 10.1 mm
- net /K9: track 12.5 -> 11.9 mm
- net /K1: track 8.74 -> 8.21 mm
- net /K7: track 8.72 -> 8.18 mm
- net /A: track 8.77 -> 8.24 mm
Other:
- board text added: "2023"
- board text added: "A"
- board text added: "James Gallagher"
- board text added: "dp"
- board text added: "front"
- board text added: "k0"
- board text added: "k1"
- board text added: "k2"
- board text added: "k3"
- board text added: "k4"
- board text added: "k5"
- board text added: "k6"
- board text added: "k7"
- board text added: "k8"
- board text added: "k9"
