File: PCB/Z573M-tube/Z573M-tube.kicad_sch (KiCad schematic)
At the start: 3 parts, among them J1 6-pin-header, J2 6-pin-header

Commit message: New board, v 2.0, with gerber files
Parts:
- V1: footprint nixie-footprints:Z57xM-v1 -> nixie-footprints:Z57xM-v3-HV
Changed lines of the file:
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@@
       (effects (font (size 1.27 1.27)) (justify left))
     )
-    (property "Footprint" "nixie-footprints:Z57xM-v1" (id 2) (at 148.59 95.25 0)
+    (property "Footprint" "nixie-footprints:Z57xM-v3-HV" (id 2) (at 148.59 95.25 0)
       (effects (font (size 1.27 1.27)) hide)
     )
@@
     )
     (path "/5d4c135e-579a-4b9e-b225-7fc16597da71"
-      (reference "V1") (unit 1) (value "Z57xM") (footprint "nixie-footprints:Z57xM-v1")
+      (reference "V1") (unit 1) (value "Z57xM") (footprint "nixie-footprints:Z57xM-v3-HV")
     )
   )
