File: PCB/nixie-2.1/nixie-2.1/nixie-2.1.kicad_pcb (KiCad board)
At the start: 2 copper layers, 167.1 x 142.7 mm, 86 parts, among them J1 Barrel_Jack_Switch, Q1 IRF730 TO220-3, Q10 MPSA92, Q11 MPSA42, Q12 MPSA42, Q13 MPSA42, Q14 MPSA42, Q2 MPSA92, Q3 MPSA92, Q4 MPSA92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

Commit message: Update version info on board
Other:
- board text added: "Nixie 2.1 4/23/23 Version 0.1"
- board text removed: "Nixie 2.1 4/23/23 Board 0.1"
Changed lines of the file:
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@@
   (gr_line (start 182.372 19.812) (end 182.372 162.56) (layer "Margin") (width 0.15))
   (gr_line (start 15.24 19.812) (end 182.372 19.812) (layer "Margin") (width 0.15))
-  (gr_text "Nixie 2.1\n4/23/23\nBoard 0.1" (at 166.624 157.48) (layer "F.SilkS")
+  (gr_text "Nixie 2.1\n4/23/23\nVersion 0.1" (at 166.624 157.48) (layer "F.SilkS")
     (effects (font (size 1 1) (thickness 0.15)))
   )

Commit message: hacking
Parts:
- added REF**: Polarity_Center_Positive_6mm_SilkScreen, Symbol:Polarity_Center_Positive_6mm_SilkScreen, F.Cu at (164.6, 41.1)
Other:
- board text added: "James Gallagher Nixie 2.1 04/23/23 Version 0.1"
- board text removed: "James Gallagher Nixie 2.1 04/23/23 Board 0.1"

Commit message: updates
Parts:
- removed REF**: Polarity_Center_Positive_6mm_SilkScreen, Symbol:Polarity_Center_Positive_6mm_SilkScreen
- removed REF**: OSHW-Logo2_7.3x6mm_Copper, Symbol:OSHW-Logo2_7.3x6mm_Copper
- removed REF**: KiCad-Logo2_5mm_Copper, Symbol:KiCad-Logo2_5mm_Copper
- CR1: value MUR 160 G -> MUR160G
- Q10, Q12, Q13, Q2, Q3, Q4, Q5, Q6, Q7, Q8, Q9: footprint Package_TO_SOT_THT:TO-92L_HandSolder -> nixie-2.1-footprints:TO-92_HandSolder
- Q11, Q14: footprint Package_TO_SOT_THT:TO-92L_HandSolder -> Package_TO_SOT_THT:TO-92_HandSolder
- R6: value 10K -> 10K_Trimmer
Routing:
- net GND: track 0.88 -> 2.44 mm, vias 0 -> 1
- net SDA: track 41.7 -> 43.2 mm
