File: PCB/nixie-2.1/nixie-2.1/nixie_2_ps.kicad_sch (KiCad schematic)
At the start: 20 parts, among them J1 Barrel_Jack_Switch, Q1 IRF730 TO220-3, U1 LM317_TO-220

Commit message: updates
Other:
- moved on the sheet: C3
