File: PCB/nixie-2.1/nixie-2.1/nixies_2.1_display.kicad_sch (KiCad schematic)
At the start: 51 parts, among them Q10 MPSA92, Q11 MPSA42, Q12 MPSA42, Q13 MPSA42, Q14 MPSA42, Q2 MPSA92, Q3 MPSA92, Q4 MPSA92, Q5 MPSA42, Q6 MPSA42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

Commit message: updates
Parts:
- Q10, Q12, Q13, Q2, Q3, Q4, Q5, Q6, Q7, Q8, Q9: footprint Package_TO_SOT_THT:TO-92_Inline -> nixie-2.1-footprints:TO-92_HandSolder
- Q11, Q14: footprint Package_TO_SOT_THT:TO-92_Inline -> Package_TO_SOT_THT:TO-92_HandSolder
