File: PCB/nixie-2.1/nixie-2.1.kicad_pcb (KiCad board)
At the start: 2 copper layers, 167.1 x 142.7 mm, 84 parts, among them J1 Barrel_Jack_Switch, Q1 IRF730 TO220-3, Q10 MPSA92, Q11 MPSA42, Q12 MPSA42, Q13 MPSA42, Q14 MPSA42, Q2 MPSA92, Q3 MPSA92, Q4 MPSA92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

Commit message: Reorganization
Parts:
- added G***: LOGO, nixie-2.1-footprints:High-voltage-25mm-v2-with-text, F.Cu at (117.3, 95.0)
- added G***: LOGO, nixie-2.1-footprints:High-voltage-25mm-v2-with-text, F.Cu at (66.0, 95.0)
- added G***: LOGO, nixie-2.1-footprints:QR-code-jhrg-nixie-2, B.Cu at (56.9, 59.9)
- added REF**: High-Voltage-25mm, nixie-2.1-footprints:High-Voltage-25mm, F.Cu at (116.8, 71.6)
- added REF**: OSHW-Logo2_9.8x8mm_SilkScreen, Symbol:OSHW-Logo2_9.8x8mm_SilkScreen, F.Cu at (172.7, 146.3)
- added REF**: Polarity_Center_Positive_6mm_SilkScreen, Symbol:Polarity_Center_Positive_6mm_SilkScreen, F.Cu at (164.6, 41.1)
Other:
- board text added: "locked"
- board text removed: "James Gallagher Nixie 2.1 04/23/23 Version 0.1"

Commit message: New display-only board
Parts:
- removed the REF** at (116.8, 71.6)
Connections:
- Q10 pad 1: Net-(Q10-E) -> HV
- Q10 pad 3: HV -> Net-(Q10-C)
- Q2 pad 1: Net-(Q2-E) -> HV
- Q2 pad 3: HV -> Net-(Q2-C)
- Q3 pad 1: Net-(Q3-E) -> HV
- Q3 pad 3: HV -> Net-(Q3-C)
- Q4 pad 1: Net-(Q4-E) -> HV
- Q4 pad 3: HV -> Net-(Q4-C)
- Q8 pad 1: Net-(Q8-E) -> HV
- Q8 pad 3: HV -> Net-(Q8-C)
- Q9 pad 1: Net-(Q9-E) -> HV
- Q9 pad 3: HV -> Net-(Q9-C)
- R13 pad 1: Net-(Q2-E) -> Net-(Q2-C)
- R14 pad 1: Net-(Q3-E) -> Net-(Q3-C)
- R15 pad 1: Net-(Q4-E) -> Net-(Q4-C)
- R28 pad 1: Net-(Q8-E) -> Net-(Q8-C)
- R29 pad 1: Net-(Q9-E) -> Net-(Q9-C)
- R30 pad 1: Net-(Q10-E) -> Net-(Q10-C)
Routing:
- net HV: track 235.9 -> 258.5 mm
- net Net-(Q9-C): track 0.00 -> 10.00 mm
- net Net-(Q10-C): track 0.00 -> 9.36 mm
- net Net-(Q8-C): track 0.00 -> 9.36 mm
- net Net-(Q3-C): track 0.00 -> 9.36 mm
- net Net-(Q4-C): track 0.00 -> 9.09 mm
- net Net-(Q9-E): track 8.95 -> 0.00 mm
- net Net-(Q2-C): track 0.00 -> 8.88 mm
- net Net-(Q10-E): track 8.31 -> 0.00 mm
- net Net-(Q8-E): track 8.31 -> 0.00 mm
- net Net-(Q3-E): track 8.31 -> 0.00 mm
- net Net-(Q4-E): track 8.04 -> 0.00 mm
- net Net-(Q2-E): track 7.83 -> 0.00 mm
Other:
- board text added: "Nixie 2.1 05/07/23 Version 0.2"
- board text removed: "Nixie 2.1 4/23/23 Version 0.1"
